Commit message: the mpc ros max time is easy to be long

File: lxfr_description/urdf/include/lxfr_v1.urdf.xacro (robot description, xacro)
@@ -133,8 +133,11 @@
         </material>
       </visual>
-      <collision>
-        <origin xyz="${lxfr_act_wheel_dx} 0 0" rpy="0 0 0" />
-        <geometry>
-          <mesh filename="package://lxfr_description/meshes/lxfr_base.stl"/>
+      <!-- modified by yq for robot_body_filter -->
+      <collision>
+      <origin xyz="0.025 -0.46174 0.261" rpy="0 0 ${pi}" />
+        <!-- <origin xyz="${lxfr_act_wheel_dx} 0 0" rpy="0 0 0" />  -->
+        <geometry>
+         <mesh filename="package://lxfr_description/meshes/base_link.STL"/>
+          <!-- <mesh filename="package://lxfr_description/meshes/lxfr_base.stl"/> -->
         </geometry>
       </collision>

File: mue_description/urdf/lxfr_v1.urdf.xacro (robot description, xacro)
@@ -151,15 +151,12 @@
         </material>
       </visual>
-      <collision>
-        <origin xyz="${lxfr_act_wheel_dx} 0 0" rpy="0 0 0" />
-        <geometry>
-          <mesh filename="package://lxfr_description/meshes/lxfr_base.stl"/>
-        </geometry>
-                  <friction>
-            <ode>
-                <mu>2</mu>
-                <mu2>2</mu2>
-            </ode>
-          </friction>
+      <!-- modified by yq for robot_body_filter -->
+      <collision>
+      <origin xyz="0.025 -0.46174 0.261" rpy="0 0 ${pi}" />
+        <!-- <origin xyz="${lxfr_act_wheel_dx} 0 0" rpy="0 0 0" />  -->
+        <geometry>
+         <mesh filename="package://lxfr_description/meshes/base_link.STL"/>
+          <!-- <mesh filename="package://lxfr_description/meshes/lxfr_base.stl"/> -->
+        </geometry>
       </collision>
     </link>
